File: psnee.kicad_pcb (KiCad board)
At the start: 2 copper layers, 21 x 36 mm, 10 parts, among them IC1 ATTINY45, P1 CONN_ICSP

Commit message: pcb for v2.0
Parts:
- removed a18, d2, dat, gate, gnd, lid, vcc: wire_pad_2.5_5mm_single, psnee:wire_pad_2.5_5mm_single
- added 1: wire_pad_2.5_5mm_single, psnee:wire_pad_2.5_5mm_single, F.Cu at (163.2, 52.9)
- added 2: wire_pad_2.5_5mm_single, psnee:wire_pad_2.5_5mm_single, F.Cu at (159.7, 52.9)
- added 3: wire_pad_2.5_5mm_single, psnee:wire_pad_2.5_5mm_single, F.Cu at (156.2, 52.9)
- added 4: wire_pad_2.5_5mm_single, psnee:wire_pad_2.5_5mm_single, F.Cu at (152.7, 52.9)
- added 5: wire_pad_2.5_5mm_single, psnee:wire_pad_2.5_5mm_single, F.Cu at (149.2, 52.9)
- added 6: wire_pad_2.5_5mm_single, psnee:wire_pad_2.5_5mm_single, F.Cu at (145.7, 52.9)
- added 7: wire_pad_2.5_5mm_single, psnee:wire_pad_2.5_5mm_single, F.Cu at (142.2, 52.9)
- added 8: wire_pad_2.5_5mm_single, psnee:wire_pad_2.5_5mm_single, F.Cu at (138.7, 52.9)
- added C1: 100nF, Capacitors_ThroughHole:C_Disc_D6_P5, F.Cu at (139.5, 67.1)
- added C2: 100uF, Capacitors_ThroughHole:C_Radial_D5_L11_P2, F.Cu at (141.3, 60.8)
- IC1: value ATTINY45 -> attiny45
- P1: value CONN_ICSP -> header
- moved IC1 60.5 mm to (128.0, 68.0), turned to 90 degrees
- moved D1 29.6 mm to (147.0, 68.4), turned to 0 degrees
- moved P1 25.0 mm to (160.1, 62.7), turned to 0 degrees
Connections:
- net /data renamed /5
- net /gate renamed /6
- net /lid renamed /7
- net Net-(IC1-Pad1) renamed /1
- IC1 pad 2: /biosA18 -> /2
- IC1 pad 3: /biosD2 -> /3
Routing:
- net /2: track 0.00 -> 58.0 mm, vias 0 -> 1
- net /3: track 0.00 -> 54.7 mm, vias 0 -> 1
- net /1: track 34.4 -> 78.8 mm
- net /6: track 68.6 -> 34.7 mm
- net /biosD2: track 28.2 -> 0.00 mm
- net /biosA18: track 24.6 -> 0.00 mm
- net VCC: track 3.81 -> 26.5 mm, vias 1 -> 0
- net Net-(C1-Pad1): track 30.8 -> 48.0 mm
- net /7: track 46.6 -> 38.3 mm
- net /5: track 29.6 -> 37.1 mm
- net GND: track 3.30 -> 2.79 mm
- added copper zone on B.Cu, net GND
- removed copper zone on B.Cu, net VCC
Other:
- board size 21 x 36 mm -> 40 x 20 mm
- net class Default: clearance 0.254 -> 0.1524; trace_width 0.254 -> 0.1524; via_dia 0.6858 -> 0.508; via_drill 0.3302 -> 0.254
- rule trace_clearance: 0.254 -> 0.1524
- rule via_min_drill: 0.3302 -> 0.254
- rule via_min_size: 0.6858 -> 0.4
- board text removed: "PSNee[t] @komidore64 v1.0"

Commit message: added text for pcb v2
Other:
- board text added: "PSNee[t] @komidore64 v2"
Changed lines of the file:
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@@
     (area 123.2186 48.0081 173.041448 71.5469)
     (thickness 1.6)
-    (drawings 4)
+    (drawings 5)
     (tracks 66)
     (zones 0)
@@
   )
   (page A4)
+  (title_block
+    (title PSNee[t])
+    (date 2018-03-13)
+    (rev v2)
+  )
   (layers
     (0 F.Cu signal)
@@
     (pad_to_mask_clearance 0)
     (aux_axis_origin 0 0)
-    (visible_elements FFFEFF7F)
+    (visible_elements FFFEFFFF)
     (pcbplotparams
       (layerselection 0x00030_80000001)
@@
       (net 3 VCC))
   )
+  (gr_text "PSNee[t]\n@komidore64\nv2" (at 163.703 54.8005 -360) (layer B.SilkS)
+    (effects (font (size 1.5 1.5) (thickness 0.3)) (justify left mirror))
+  )
   (gr_line (start 165 50) (end 125 50) (angle 90) (layer Edge.Cuts) (width 0.1))

Commit message: add oshw logo
Parts:
- added REF**: Symbol_OSHW-Logo_SilkScreen, Symbols:Symbol_OSHW-Logo_SilkScreen, B.Cu at (150.7, 61.5)
Changed lines of the file:
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@@
     (tracks 66)
     (zones 0)
-    (modules 13)
+    (modules 14)
     (nets 10)
   )
@@
     (pad_to_mask_clearance 0)
     (aux_axis_origin 0 0)
-    (visible_elements FFFEFFFF)
+    (visible_elements FFFEFF7F)
     (pcbplotparams
       (layerselection 0x00030_80000001)
@@
       (net 3 VCC))
   )
-  (gr_text "PSNee[t]\n@komidore64\nv2" (at 163.703 54.8005 -360) (layer B.SilkS)
+  (module Symbols:Symbol_OSHW-Logo_SilkScreen (layer B.Cu)
+    (at 150.6855 61.5315 180)
+    (descr "Symbol, OSHW-Logo, Silk Screen,")
+    (tags "Symbol, OSHW-Logo, Silk Screen,")
+    (fp_text reference REF** (at 0.09906 4.38912 180) (layer B.SilkS) hide
+      (effects (font (size 1 1) (thickness 0.15)) (justify mirror))
+    )
+    (fp_text value Symbol_OSHW-Logo_SilkScreen (at 0.30988 -6.56082 180) (layer B.Fab)
+      (effects (font (size 1 1) (thickness 0.15)) (justify mirror))
+    )
+    (fp_line (start 1.66878 -2.68986) (end 2.02946 -4.16052) (layer B.SilkS) (width 0.15))
+    (fp_line (start 2.02946 -4.16052) (end 2.30886 -3.0988) (layer B.SilkS) (width 0.15))
+    (fp_line (start 2.30886 -3.0988) (end 2.61874 -4.17068) (layer B.SilkS) (width 0.15))
+    (fp_line (start 2.61874 -4.17068) (end 2.9591 -2.72034) (layer B.SilkS) (width 0.15))
+    (fp_line (start 0.24892 -3.38074) (end 1.03886 -3.37058) (layer B.SilkS) (width 0.15))
+    (fp_line (start 1.03886 -3.37058) (end 1.04902 -3.38074) (layer B.SilkS) (width 0.15))
+    (fp_line (start 1.04902 -3.38074) (end 1.04902 -3.37058) (layer B.SilkS) (width 0.15))
+    (fp_line (start 1.08966 -2.65938) (end 1.08966 -4.20116) (layer B.SilkS) (width 0.15))
+    (fp_line (start 0.20066 -2.64922) (end 0.20066 -4.21894) (layer B.SilkS) (width 0.15))
+    (fp_line (start 0.20066 -4.21894) (end 0.21082 -4.20878) (layer B.SilkS) (width 0.15))
+    (fp_line (start -0.35052 -2.75082) (end -0.70104 -2.66954) (layer B.SilkS) (width 0.15))
+    (fp_line (start -0.70104 -2.66954) (end -1.02108 -2.65938) (layer B.SilkS) (width 0.15))
+    (fp_line (start -1.02108 -2.65938) (end -1.25984 -2.86004) (layer B.SilkS) (width 0.15))
+    (fp_line (start -1.25984 -2.86004) (end -1.29032 -3.12928) (layer B.SilkS) (width 0.15))
+    (fp_line (start -1.29032 -3.12928) (end -1.04902 -3.37058) (layer B.SilkS) (width 0.15))
+    (fp_line (start -1.04902 -3.37058) (end -0.6604 -3.50012) (layer B.SilkS) (width 0.15))
+    (fp_line (start -0.6604 -3.50012) (end -0.48006 -3.66014) (layer B.SilkS) (width 0.15))
+    (fp_line (start -0.48006 -3.66014) (end -0.43942 -3.95986) (layer B.SilkS) (width 0.15))
+    (fp_line (start -0.43942 -3.95986) (end -0.67056 -4.18084) (layer B.SilkS) (width 0.15))
+    (fp_line (start -0.67056 -4.18084) (end -0.9906 -4.20878) (layer B.SilkS) (width 0.15))
+    (fp_line (start -0.9906 -4.20878) (end -1.34112 -4.09956) (layer B.SilkS) (width 0.15))
+    (fp_line (start -2.37998 -2.64922) (end -2.6289 -2.66954) (layer B.SilkS) (width 0.15))
+    (fp_line (start -2.6289 -2.66954) (end -2.8702 -2.91084) (layer B.SilkS) (width 0.15))
+    (fp_line (start -2.8702 -2.91084) (end -2.9591 -3.40106) (layer B.SilkS) (width 0.15))
+    (fp_line (start -2.9591 -3.40106) (end -2.93116 -3.74904) (layer B.SilkS) (width 0.15))
+    (fp_line (start -2.93116 -3.74904) (end -2.7305 -4.06908) (layer B.SilkS) (width 0.15))
+    (fp_line (start -2.7305 -4.06908) (end -2.47904 -4.191) (layer B.SilkS) (width 0.15))
+    (fp_line (start -2.47904 -4.191) (end -2.16916 -4.11988) (layer B.SilkS) (width 0.15))
+    (fp_line (start -2.16916 -4.11988) (end -1.95072 -3.93954) (layer B.SilkS) (width 0.15))
+    (fp_line (start -1.95072 -3.93954) (end -1.8796 -3.4798) (layer B.SilkS) (width 0.15))
+    (fp_line (start -1.8796 -3.4798) (end -1.9304 -3.07086) (layer B.SilkS) (width 0.15))
+    (fp_line (start -1.9304 -3.07086) (end -2.03962 -2.78892) (layer B.SilkS) (width 0.15))
+    (fp_line (start -2.03962 -2.78892) (end -2.4003 -2.65938) (layer B.SilkS) (width 0.15))
+    (fp_line (start -1.78054 -0.92964) (end -2.03962 -1.49098) (layer B.SilkS) (width 0.15))
+    (fp_line (start -2.03962 -1.49098) (end -1.50114 -2.00914) (layer B.SilkS) (width 0.15))
+    (fp_line (start -1.50114 -2.00914) (end -0.98044 -1.7399) (layer B.SilkS) (width 0.15))
+    (fp_line (start -0.98044 -1.7399) (end -0.70104 -1.89992) (layer B.SilkS) (width 0.15))
+    (fp_line (start 0.73914 -1.8796) (end 1.06934 -1.6891) (layer B.SilkS) (width 0.15))
+    (fp_line (start 1.06934 -1.6891) (end 1.50876 -2.0193) (layer B.SilkS) (width 0.15))
+    (fp_line (start 1.50876 -2.0193) (end 1.9812 -1.52908) (layer B.SilkS) (width 0.15))
+    (fp_line (start 1.9812 -1.52908) (end 1.69926 -1.04902) (layer B.SilkS) (width 0.15))
+    (fp_line (start 1.69926 -1.04902) (end 1.88976 -0.57912) (layer B.SilkS) (width 0.15))
+    (fp_line (start 1.88976 -0.57912) (end 2.49936 -0.39116) (layer B.SilkS) (width 0.15))
+    (fp_line (start 2.49936 -0.39116) (end 2.49936 0.28956) (layer B.SilkS) (width 0.15))
+    (fp_line (start 2.49936 0.28956) (end 1.94056 0.42926) (layer B.SilkS) (width 0.15))
+    (fp_line (start 1.94056 0.42926) (end 1.7399 1.00076) (layer B.SilkS) (width 0.15))
+    (fp_line (start 1.7399 1.00076) (end 2.00914 1.47066) (layer B.SilkS) (width 0.15))
+    (fp_line (start 2.00914 1.47066) (end 1.53924 1.9812) (layer B.SilkS) (width 0.15))
+    (fp_line (start 1.53924 1.9812) (end 1.02108 1.71958) (layer B.SilkS) (width 0.15))
+    (fp_line (start 1.02108 1.71958) (end 0.55118 1.92024) (layer B.SilkS) (width 0.15))
+    (fp_line (start 0.55118 1.92024) (end 0.381 2.46126) (layer B.SilkS) (width 0.15))
+    (fp_line (start 0.381 2.46126) (end -0.30988 2.47904) (layer B.SilkS) (width 0.15))
+    (fp_line (start -0.30988 2.47904) (end -0.5207 1.9304) (layer B.SilkS) (width 0.15))
+    (fp_line (start -0.5207 1.9304) (end -0.9398 1.76022) (layer B.SilkS) (width 0.15))
+    (fp_line (start -0.9398 1.76022) (end -1.49098 2.02946) (layer B.SilkS) (width 0.15))
+    (fp_line (start -1.49098 2.02946) (end -2.00914 1.50114) (layer B.SilkS) (width 0.15))
+    (fp_line (start -2.00914 1.50114) (end -1.76022 0.96012) (layer B.SilkS) (width 0.15))
+    (fp_line (start -1.76022 0.96012) (end -1.9304 0.48006) (layer B.SilkS) (width 0.15))
+    (fp_line (start -1.9304 0.48006) (end -2.47904 0.381) (layer B.SilkS) (width 0.15))
+    (fp_line (start -2.47904 0.381) (end -2.4892 -0.32004) (layer B.SilkS) (width 0.15))
+    (fp_line (start -2.4892 -0.32004) (end -1.9304 -0.5207) (layer B.SilkS) (width 0.15))
+    (fp_line (start -1.9304 -0.5207) (end -1.7907 -0.91948) (layer B.SilkS) (width 0.15))
+    (fp_line (start 0.35052 -0.89916) (end 0.65024 -0.7493) (layer B.SilkS) (width 0.15))
+    (fp_line (start 0.65024 -0.7493) (end 0.8509 -0.55118) (layer B.SilkS) (width 0.15))
+    (fp_line (start 0.8509 -0.55118) (end 1.00076 -0.14986) (layer B.SilkS) (width 0.15))
+    (fp_line (start 1.00076 -0.14986) (end 1.00076 0.24892) (layer B.SilkS) (width 0.15))
+    (fp_line (start 1.00076 0.24892) (end 0.8509 0.59944) (layer B.SilkS) (width 0.15))
+    (fp_line (start 0.8509 0.59944) (end 0.39878 0.94996) (layer B.SilkS) (width 0.15))
+    (fp_line (start 0.39878 0.94996) (end -0.0508 1.00076) (layer B.SilkS) (width 0.15))
+    (fp_line (start -0.0508 1.00076) (end -0.44958 0.89916) (layer B.SilkS) (width 0.15))
+    (fp_line (start -0.44958 0.89916) (end -0.8509 0.55118) (layer B.SilkS) (width 0.15))
+    (fp_line (start -0.8509 0.55118) (end -1.00076 0.09906) (layer B.SilkS) (width 0.15))
+    (fp_line (start -1.00076 0.09906) (end -0.94996 -0.39878) (layer B.SilkS) (width 0.15))
+    (fp_line (start -0.94996 -0.39878) (end -0.70104 -0.70104) (layer B.SilkS) (width 0.15))
+    (fp_line (start -0.70104 -0.70104) (end -0.35052 -0.89916) (layer B.SilkS) (width 0.15))
+    (fp_line (start -0.35052 -0.89916) (end -0.70104 -1.89992) (layer B.SilkS) (width 0.15))
+    (fp_line (start 0.35052 -0.89916) (end 0.7493 -1.89992) (layer B.SilkS) (width 0.15))
+  )
+  (gr_text "PSNee[t]\n@komidore64\nv2" (at 163.703 54.8005) (layer B.SilkS)
     (effects (font (size 1.5 1.5) (thickness 0.3)) (justify left mirror))
   )
